File: elec/layout/default/lis2dh12tr.kicad_pcb (KiCad board)
At the start: 2 copper layers, 225.7 x 100.8 mm, 0 parts

Commit message: layout
Parts:
- added C1: Multilayer Ceramic Capacitors MLCC - SMD/SMT 100nF 10V 0402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, lib:C0402, F.Cu at (133.2, 93.3)
- added U1: , lib:LGA-12_L2.0-W2.0-P0.50-BL, F.Cu at (133.3, 95.2)
Routing:
- net vcc: track 0.00 -> 3.38 mm
- net gnd: track 0.00 -> 2.82 mm
Changed lines of the file:
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@@
   )
   (net 0 "")
+  (net 1 "int1")
+  (net 2 "int2")
+  (net 3 "gnd")
+  (net 4 "sda_sdi_sdo")
+  (net 5 "sdo_sa0")
+  (net 6 "scl_spc")
+  (net 7 "vcc")
+  (footprint "lib:LGA-12_L2.0-W2.0-P0.50-BL" (layer "F.Cu")
+    (at 133.255 95.245)
+    (attr smd)
+    (fp_text reference "U1" (at 0 -4.88) (layer "F.SilkS")
+        (effects (font (size 1 1) (thickness 0.15)))
+    )
+    (fp_text value "" (at 0 4.88) (layer "F.Fab")
+        (effects (font (size 1 1) (thickness 0.15)))
+    )
+    (fp_text user "${REFERENCE}" (at 0 0) (layer "F.Fab")
+        (effects (font (size 1 1) (thickness 0.15)))
+    )
+    (fp_line (start -1.27 -1.14) (end -1.27 -0.51)
+      (stroke (width 0.1) (type solid)) (layer "F.SilkS"))
+    (fp_line (start -1.27 0.51) (end -1.27 1.14)
+      (stroke (width 0.1) (type solid)) (layer "F.SilkS"))
+    (fp_line (start -1.27 1.14) (end -1.04 1.14)
+      (stroke (width 0.1) (type solid)) (layer "F.SilkS"))
+    (fp_line (start -1.01 -1.14) (end -1.27 -1.14)
+      (stroke (width 0.1) (type solid)) (layer "F.SilkS"))
+    (fp_line (start 1.02 -1.14) (end 1.27 -1.14)
+      (stroke (width 0.1) (type solid)) (layer "F.SilkS"))
+    (fp_line (start 1.27 -1.14) (end 1.27 -0.51)
+      (stroke (width 0.1) (type solid)) (layer "F.SilkS"))
+    (fp_line (start 1.27 0.51) (end 1.27 1.14)
+      (stroke (width 0.1) (type solid)) (layer "F.SilkS"))
+    (fp_line (start 1.27 1.14) (end 1.02 1.14)
+      (stroke (width 0.1) (type solid)) (layer "F.SilkS"))
+    (fp_circle (center -0.75 1.46) (end -0.68 1.46)
+      (stroke (width 0.15) (type solid)) (fill none) (layer "F.SilkS"))
+    (fp_circle (center -0.75 1.29) (end -0.68 1.29)
+      (stroke (width 0.15) (type solid)) (fill none) (layer "Cmts.User"))
+    (fp_circle (center -1 1) (end -0.97 1)
+      (stroke (width 0.06) (type solid)) (fill none) (layer "F.Fab"))
+    (pad "1" smd rect (at -0.75 0.88) (size 0.28 0.5) (layers "F.Cu" "F.Paste" "F.Mask")
+      (net 6 "scl_spc") (pintype "stereo"))
+    (pad "2" smd rect (at -0.25 0.88) (size 0.28 0.5) (layers "F.Cu" "F.Paste" "F.Mask")
+      (net 7 "vcc") (pintype "stereo"))
+    (pad "3" smd rect (at 0.25 0.88) (size 0.28 0.5) (layers "F.Cu" "F.Paste" "F.Mask")
+      (net 5 "sdo_sa0") (pintype "stereo"))
+    (pad "4" smd rect (at 0.75 0.88) (size 0.28 0.5) (layers "F.Cu" "F.Paste" "F.Mask")
+      (net 4 "sda_sdi_sdo") (pintype "stereo"))
+    (pad "5" smd rect (at 0.88 0.25) (size 0.5 0.28) (layers "F.Cu" "F.Paste" "F.Mask")
+      (net 3 "gnd") (pintype "stereo"))
+    (pad "6" smd rect (at 0.88 -0.25) (size 0.5 0.28) (layers "F.Cu" "F.Paste" "F.Mask")
+      (net 3 "gnd") (pintype "stereo"))
+    (pad "7" smd rect (at 0.75 -0.88) (size 0.28 0.5) (layers "F.Cu" "F.Paste" "F.Mask")
+      (net 3 "gnd") (pintype "stereo"))
+    (pad "8" smd rect (at 0.25 -0.88) (size 0.28 0.5) (layers "F.Cu" "F.Paste" "F.Mask")
+      (net 3 "gnd") (pintype "stereo"))
+    (pad "9" smd rect (at -0.25 -0.88) (size 0.28 0.5) (layers "F.Cu" "F.Paste" "F.Mask")
+      (net 7 "vcc") (pintype "stereo"))
+    (pad "10" smd rect (at -0.75 -0.88) (size 0.28 0.5) (layers "F.Cu" "F.Paste" "F.Mask")
+      (net 7 "vcc") (pintype "stereo"))
+    (pad "11" smd rect (at -0.88 -0.25) (size 0.5 0.28) (layers "F.Cu" "F.Paste" "F.Mask")
+      (net 2 "int2") (pintype "stereo"))
+    (pad "12" smd rect (at -0.88 0.25) (size 0.5 0.28) (layers "F.Cu" "F.Paste" "F.Mask")
+      (net 1 "int1") (pintype "stereo"))
+    (model "/Users/narayanpowderly/Documents/atopile-workspace/the-everything-sensor/.ato/modules/lis2dh12tr/elec/footprints/footprints.3dshapes/LGA-12_L2.0-W2.0-H1.0-P0.50.wrl"
+      (offset (xyz 0 0 -0))
+      (scale (xyz 1 1 1))
+      (rotate (xyz 0 0 270))
+    )
+  )
+  (footprint "lib:C0402" (layer "F.Cu")
+    (at 133.240113 93.346641)
+    (descr "Capacitor SMD 0402 (1005 Metric), square (rectangular) end terminal, IPC_7351 nominal, (Body size source: IPC-SM-782 page 76, https://www.pcb-3d.com/wordpress/wp-content/uploads/ipc-sm-782a_amendment_1_and_2.pdf), generated with kicad-footprint-generator")
+    (tags "capacitor")
+    (attr smd)
+    (fp_text reference "C1" (at 0 -1.16) (layer "F.SilkS")
+        (effects (font (size 1 1) (thickness 0.15)))
+    )
+    (fp_text value "Multilayer Ceramic Capacitors MLCC - SMD/SMT 100nF 10V 0402 RoHS" (at 0 1.16) (layer "F.Fab")
+        (effects (font (size 1 1) (thickness 0.15)))
+    )
+    (fp_text user "${REFERENCE}" (at 0 0) (layer "F.Fab")
+        (effects (font (size 0.25 0.25) (thickness 0.04)))
+    )
+    (fp_line (start -0.107836 -0.36) (end 0.107836 -0.36)
+      (stroke (width 0.12) (type solid)) (layer "F.SilkS"))
+    (fp_line (start -0.107836 0.36) (end 0.107836 0.36)
+      (stroke (width 0.12) (type solid)) (layer "F.SilkS"))
+    (fp_line (start -0.91 -0.46) (end 0.91 -0.46)
+      (stroke (width 0.05) (type solid)) (layer "F.CrtYd"))
+    (fp_line (start -0.91 0.46) (end -0.91 -0.46)
+      (stroke (width 0.05) (type solid)) (layer "F.CrtYd"))
+    (fp_line (start 0.91 -0.46) (end 0.91 0.46)
+      (stroke (width 0.05) (type solid)) (layer "F.CrtYd"))
+    (fp_line (start 0.91 0.46) (end -0.91 0.46)
+      (stroke (width 0.05) (type solid)) (layer "F.CrtYd"))
+    (fp_line (start -0.5 -0.25) (end 0.5 -0.25)
+      (stroke (width 0.1) (type solid)) (layer "F.Fab"))
+    (fp_line (start -0.5 0.25) (end -0.5 -0.25)
+      (stroke (width 0.1) (type solid)) (layer "F.Fab"))
+    (fp_line (start 0.5 -0.25) (end 0.5 0.25)
+      (stroke (width 0.1) (type solid)) (layer "F.Fab"))
+    (fp_line (start 0.5 0.25) (end -0.5 0.25)
+      (stroke (width 0.1) (type solid)) (layer "F.Fab"))
+    (pad "1" smd roundrect (at -0.48 0) (size 0.56 0.62) (layers "F.Cu" "F.Paste" "F.Mask") (roundrect_rratio 0.25)
+      (net 7 "vcc") (pintype "stereo"))
+    (pad "2" smd roundrect (at 0.48 0) (size 0.56 0.62) (layers "F.Cu" "F.Paste" "F.Mask") (roundrect_rratio 0.25)
+      (net 3 "gnd") (pintype "stereo"))
+    (model "${KICAD6_3DMODEL_DIR}/Capacitor_SMD.3dshapes/C_0402_1005Metric.wrl"
+      (offset (xyz 0 0 0))
+      (scale (xyz 1 1 1))
+      (rotate (xyz 0 0 0))
+    )
+  )
   (gr_circle (center 225.62 81.79) (end 227.32 81.79)
     (stroke (width 0.1) (type solid)) (fill none) (layer "Edge.Cuts"))
@@
       (xy 69.100734 49.778315)
     )
-    (stroke (width 0) (type solid)) (fill none) (layer "Edge.Cuts"))
+    (stroke (width 0.1) (type solid)) (fill none) (layer "Edge.Cuts"))
   (gr_arc (start 261.62 113.79) (mid 260.448427 116.618427) (end 257.62 117.79)
     (stroke (width 0.1) (type solid)) (layer "Edge.Cuts"))
@@
     (effects (font (size 2 2) (thickness 0.1)) (justify left bottom))
   )
+  (segment (start 134.135 94.995) (end 134.135 95.495) (width 0.25) (layer "F.Cu") (net 3))
+  (segment (start 133.720113 93.346641) (end 133.720113 93.677419) (width 0.25) (layer "F.Cu") (net 3))
+  (segment (start 134.005 94.365) (end 133.505 94.365) (width 0.25) (layer "F.Cu") (net 3))
+  (segment (start 134.005 94.865) (end 134.135 94.995) (width 0.25) (layer "F.Cu") (net 3))
+  (segment (start 134.005 94.365) (end 134.005 94.865) (width 0.25) (layer "F.Cu") (net 3))
+  (segment (start 133.720113 93.677419) (end 134.005 93.962306) (width 0.25) (layer "F.Cu") (net 3))
+  (segment (start 134.005 93.962306) (end 134.005 94.365) (width 0.25) (layer "F.Cu") (net 3))
+  (segment (start 133.005 93.774071) (end 133.005 94.365) (width 0.25) (layer "F.Cu") (net 7))
+  (segment (start 132.505 94.365) (end 133.005 94.365) (width 0.25) (layer "F.Cu") (net 7))
+  (segment (start 132.760113 93.346641) (end 132.760113 93.529184) (width 0.25) (layer "F.Cu") (net 7))
+  (segment (start 133.005 96.125) (end 133.005 94.365) (width 0.25) (layer "F.Cu") (net 7))
+  (segment (start 132.760113 93.529184) (end 133.005 93.774071) (width 0.25) (layer "F.Cu") (net 7))
   (group "" (id 6c1ef9f7-0f34-47bb-ac1a-76df23fb396e)
     (members
